Commit message: Navigation and GPS

File: ws_urc/src/robot_description/urdf/sensors/imu.urdf.xacro (robot description, xacro)
@@ -5,5 +5,7 @@
       <parent link="base_link"/>
       <child link="imu_link"/>
+      <!-- Might be error here if imu heading doesn't align with base_link -->
       <origin xyz="0 0 0" rpy="0 0 0"/>
+      <!-- we assume the robot is equipped with an IMU that can accurately measure absolute orientation following the ENU convention, meaning it will output zero yaw when facing east and +90 degrees when facing north. -->
     </joint>
     <gazebo>

File: ws_urc/src/robot_description/urdf/sensors/plugins.urdf.xacro (robot description, xacro)
@@ -7,3 +7,9 @@
     </plugin>
   </gazebo>
+  <gazebo>
+    <plugin
+      filename="gz-sim-navsat-system"
+      name="gz::sim::systems::NavSat">
+    </plugin>
+  </gazebo>
 </robot>

File: ws_urc/src/robot_description/urdf/srp.urdf.xacro (robot description, xacro)
@@ -9,4 +9,5 @@
   <xacro:include filename="$(find robot_description)/urdf/sensors/depth_sensor.urdf.xacro" />
   <xacro:include filename="$(find robot_description)/urdf/ackermann.urdf.xacro" />
+  <xacro:include filename="$(find robot_description)/urdf/sensors/gps.urdf.xacro" />
   <xacro:base
     length="${base_length}"
@@ -93,4 +94,7 @@
     <xacro:insert_block name="depth_sensor_pose" />
   </xacro:depth_sensor>
+  <xacro:gps_sensor>
+    <xacro:insert_block name="gps_pose" />
+  </xacro:gps_sensor>
   <xacro:ackermann_controller
     wheel_separation="${wheel_pos_y * 2}"

File: ws_urc/src/robot_description/urdf/srp_properties.urdf.xacro (robot description, xacro)
@@ -26,3 +26,6 @@
     <origin xyz="-0.065 0 0.255" rpy="0 0 0"/>
   </xacro:property>
+  <xacro:property name="gps_pose">
+    <origin xyz="0.1 0 0.2" rpy="0 0 0"/>
+  </xacro:property>
 </robot>
